File: skibidi-usb-hub.kicad_sch (KiCad schematic)
At the start: 0 parts

Commit message: finished schematic siuuuuu
Parts:
- added C1, C19, C21, C23, C27, C29, C3, C31, C7: 100n, Capacitor_SMD:C_0402_1005Metric, symbol Device:C
- added C10, C12, C14, C16, C18, C2, C20, C22, C24, C26, C28, C30, C32, C33, C34, C35, C36, C4, C9: 1u, Capacitor_SMD:C_0402_1005Metric, symbol Device:C
- added C11, C13, C15, C17, C25, C8: 100u, Capacitor_SMD:C_1206_3216Metric, symbol Device:C
- added C37, C38, C39, C40: 10n, Capacitor_SMD:C_0402_1005Metric, symbol Device:C
- added C5: 10u, Capacitor_SMD:C_0603_1608Metric, symbol Device:C
- added C6: 47u, Capacitor_SMD:C_0805_2012Metric, symbol Device:C
- added JP1, JP2: SolderJumper_2_Bridged, Jumper:SolderJumper-2_P1.3mm_Bridged_RoundedPad1.0x1.5mm, symbol Jumper:SolderJumper_2_Bridged
- added R1, R3, R4: 56k, Resistor_SMD:R_0402_1005Metric, symbol Device:R
- added R2, R5: 2.49k, Resistor_SMD:R_0402_1005Metric, symbol Device:R
- added RJ1, RJ2: X12ADGWA3DY1027, easyeda2kicad:RJ45-TH_XKB_X12ADHWA3DY1027, symbol easyeda2kicad:X12ADGWA3DY1027
- added SW1, SW2: B3U-1100PM, easyeda2kicad:SW-SMD_3P-L3.0-W2.5-LS4.0, symbol easyeda2kicad:B3U-1100PM
- added T1, T2: H1102NLT_C20623173, easyeda2kicad:XFMR-SMD_H1102NLT, symbol easyeda2kicad:H1102NLT_C20623173
- added TP1, TP10, TP11, TP12, TP13, TP14, TP15, TP16, TP17, TP18, TP19, TP2, TP20, TP21, TP22, TP23, TP24, TP25, TP26, TP27, TP28, TP3, TP30, TP33, TP35, TP36, TP4, TP5, TP6, TP7, TP8, TP9: TestPoint, TestPoint:TestPoint_Pad_D2.0mm, symbol Connector:TestPoint
- added U1, U8: CH334F_C5187527, easyeda2kicad:QFN-24_L4.0-W4.0-P0.50-BL-EP2.8, symbol easyeda2kicad:CH334F_C5187527
- added U10: PJ-320A-4P DIP, easyeda2kicad:AUDIO-TH_PJ-320A-4P-DIP, symbol easyeda2kicad:PJ-320A-4PDIP
- added U2: CH217K, easyeda2kicad:SOT-23-6_L2.9-W1.6-P0.95-LS2.8-BL, symbol easyeda2kicad:CH217K
- added U3, U4, U6: GT-USB-7010ASV, easyeda2kicad:USB-C-SMD_G-SWITCH_GT-USB-7010ASV, symbol easyeda2kicad:GT-USB-7010ASV
- added U5, U7: RTL8152B-VB-CG, easyeda2kicad:QFN-24_L4.0-W4.0-P0.50-BL-EP2.0, symbol easyeda2kicad:RTL8152B-VB-CG
- added U9: HS-100B, easyeda2kicad:LQFP-48_L7.0-W7.0-P0.50-LS9.0-BL, symbol easyeda2kicad:HS-100B
- added USB1, USB2: AF 90° WJDG, easyeda2kicad:USB-A-TH_AF-WJDG, symbol easyeda2kicad:AF90°WJDG
- added X1, X2: X322516MLB4SI, easyeda2kicad:OSC-SMD_4P-L3.2-W2.5-BL, symbol easyeda2kicad:X322516MLB4SI
Connections:
- new net: TP5.1, U8.22 (LED1)
- new net: TP22.1, U9.3 (SK)
- new net: JP1.2 (B), TP10.1, U9.10 (MODE)
- new net: R2.1, U5.24 (RSET)
- new net: TP20.1, U9.1 (DR)
- new net: U1.1 (~{OVCUR}), U2.3 (~{FLAG})
- new net: U1.24 (~{PWREN}), U2.4 (~{EN})
- new net: R1.1, U2.5 (ISET)
- new net: TP3.1, U1.13 (LED3/SCL)
- new net: SW1.2, U1.16 (~{RESET}/CDP)
- new net: TP4.1, U1.21 (LED4/SDA)
- new net: TP1.1, U1.22 (LED1)
- new net: TP2.1, U1.23 (LED2)
- new net: C39.1, C40.1, T2.2, T2.7
- new net: RJ1.1, T1.16
- new net: RJ1.2, T1.14
- new net: RJ1.3, T1.11
- new net: RJ1.4, RJ1.5, RJ1.7, RJ1.8
- new net: RJ1.6, T1.9
- new net: TP35.1, U7.14 (GPIO)
- new net: R5.1, U7.24 (RSET)
- new net: C34.2, U9.7 (DREG18)
- new net: TP15.1, U9.47 (VOLDN)
- new net: TP17.1, U9.11 (LED0)
- new net: U9.13 (NC), U9.14 (NC), U9.15 (NC), U9.16 (NC), U9.18 (NC), U9.21 (NC), U9.22 (NC), U9.23 (NC), U9.24 (NC), U9.37 (NC), U9.38 (NC), U9.45 (NC), U9.46 (NC), U9.48 (NC), U9.9 (NC)
- new net: TP12.1, U9.17 (MUTEP)
- new net: TP18.1, U9.19 (LEDR)
- new net: TP21.1, U9.2 (DW)
- new net: C35.2, U9.26 (VBIAS)
- new net: C36.2, U9.27 (VREF)
- new net: U10.A, U9.28 (MICIN)
- new net: U10.B, U9.30 (LOL)
- new net: TP19.1, U9.31 (LOBS)
- new net: U10.C, U9.32 (LOR)
- new net: C32.2, U9.39 (AREG36)
- new net: TP23.1, U9.4 (CS)
- new net: TP13.1, U9.40 (MSEL)
- new net: TP14.1, U9.41 (VOLUP)
- new net: TP16.1, U9.42 (PDSW)
- new net: TP11.1, U9.5 (MUTER)
- new net: JP2.2 (B), TP9.1, U9.6 (PWRSEL)
- new net: C33.2, U9.8 (DREG33)
- new net: TP28.1, U5.19 (LANWAKEB)
- new net: TP7.1, U8.13 (LED3/SCL)
- new net: SW2.2, U8.16 (~{RESET}/CDP)
- new net: TP8.1, U8.21 (LED4/SDA)
- new net: TP6.1, U8.23 (LED2)
- new net: C37.1, C38.1, T1.2, T1.7
- new net: TP33.1, U7.20 (SPISDO)
- new net: R4.2, U7.18 (SPISDI/XTALDET)
- new net: TP36.1, U7.19 (LANWAKEB)
- new net: U7.21 (CKXTAL1), X2.1 (OSC1)
- new net: U7.22 (CKXTAL2), X2.3 (OSC2)
- new net: RJ2.1, T2.16
- new net: RJ2.2, T2.14
- new net: RJ2.3, T2.11
- new net: RJ2.4, RJ2.5, RJ2.7, RJ2.8
- new net: RJ2.6, T2.9
- new net: TP30.1, U5.20 (SPISDO)
- new net: TP27.1, U5.14 (GPIO)
- new net: R3.2, U5.18 (SPISDI/XTALDET)
- new net: U5.21 (CKXTAL1), X1.1 (OSC1)
- new net: U5.22 (CKXTAL2), X1.3 (OSC2)
- new net +1V0: C20.1, C21.1, C26.1, C27.1, U5.16 (DVDD10), U5.23 (AVDD10), U5.9 (U2VDD10), U7.16 (DVDD10), U7.23 (AVDD10), U7.9 (U2VDD10)
- new net +1V1: C22.1, C23.1, C30.1, C31.1, U5.12 (DVDD10_UPS), U7.12 (DVDD10_UPS)
- new net +3.3V: R3.1, R4.1, U5.1 (AVDD33), U5.10 (AVDD33), U5.13 (DVDD33), U7.1 (AVDD33), U7.10 (AVDD33), U7.13 (DVDD33)
- new net +5V: C12.1, C13.1, C14.1, C15.1, C16.1, C17.1, C18.1, C19.1, C24.1, C25.1, C28.1, C29.1, C7.1, C9.1, TP25.1, U2.1 (VOUT), U4.A4B9 (VBUS), U4.B4A9 (VBUS), U5.11 (VDD5), U6.A4B9 (VBUS), U6.B4A9 (VBUS), U7.11 (VDD5), U8.19 (V5), U9.29 (AVDD), U9.34 (AVDD), U9.35 (DVDD), USB1.1 (VCC), USB2.1 (VCC)
- new net D1+: U1.12 (DP1), U4.A6 (DP1), U4.B6 (DP2)
- new net D1-: U1.11 (DM1), U4.A7 (DN1), U4.B7 (DN2)
- new net D2+: U1.10 (DP2), USB1.2 (D-)
- new net D2-: U1.9 (DM2), USB1.3 (D+)
- new net D21+: U5.8 (U2DP), U8.12 (DP1)
- new net D21-: U5.7 (U2DM), U8.11 (DM1)
- new net D22+: U7.8 (U2DP), U8.10 (DP2)
- new net D22-: U7.7 (U2DM), U8.9 (DM2)
- new net D23+: U8.8 (DP3), U9.44 (USBDM)
- new net D23-: U8.7 (DM3), U9.43 (USBDP)
- new net D24+: U6.A6 (DP1), U6.B6 (DP2), U8.6 (DP4)
- new net D24-: U6.A7 (DN1), U6.B7 (DN2), U8.5 (DM4)
- new net D3+: U1.8 (DP3), USB2.2 (D-)
- new net D3-: U1.7 (DM3), USB2.3 (D+)
- new net D4+: U1.6 (DP4), U8.15 (DPU)
- new net D4-: U1.5 (DM4), U8.14 (DMU)
- new net DU+: U1.15 (DPU), U3.A6 (DP1), U3.B6 (DP2)
- new net DU-: U1.14 (DMU), U3.A7 (DN1), U3.B7 (DN2)
- new net GND: C1.2, C10.2, C11.2, C12.2, C13.2, C14.2, C15.2, C16.2, C17.2, C18.2, C19.2, C2.2, C20.2, C21.2, C22.2, C23.2, C24.2, C25.2, C26.2, C27.2, C28.2, C29.2, C3.2, C30.2, C31.2, C32.1, C33.1, C34.1, C35.1, C36.1, C37.2, C38.2, C39.2, C4.2, C40.2, C5.2, C6.2, C7.2, C8.2, C9.2, JP1.1 (A), JP2.1 (A), R1.2, R2.2, R5.2, SW1.1, SW1.3, SW2.1, SW2.3, TP26.1, U1.25 (GND), U10.D, U2.2 (GND), U3.1 (SHELL), U3.2 (SHELL), U3.3 (SHELL), U3.4 (SHELL), U3.A1B12 (GND), U3.B1A12 (GND), U4.1 (SHELL), U4.2 (SHELL), U4.3 (SHELL), U4.4 (SHELL), U4.A1B12 (GND), U4.B1A12 (GND), U5.25 (EP), U5.6 (U2GND), U6.1 (SHELL), U6.2 (SHELL), U6.3 (SHELL), U6.4 (SHELL), U6.A1B12 (GND), U6.B1A12 (GND), U7.25 (EP), U7.6 (U2GND), U8.25 (GND), U9.12 (DVSS), U9.20 (TEST), U9.25 (AVSS), U9.33 (AVSS), U9.36 (DVSS), USB1.4 (GND), USB1.5 (SHLD), USB2.4 (GND), USB2.5 (SHLD), X1.2 (GND), X1.4 (GND), X2.2 (GND), X2.4 (GND)
- new net LED0: RJ1.9, U5.15 (LED0/SPICSB)
- new net LED1: RJ1.10, U5.17 (LED1/SPISCK)
- new net LED2: RJ2.9, U7.15 (LED0/SPICSB)
- new net LED3: RJ2.10, U7.17 (LED1/SPISCK)
- new net MDI0+: T1.1, U5.2 (MDIP0)
- new net MDI0-: T1.3, U5.3 (MDIN0)
- new net MDI1+: T1.6, U5.4 (MDIP1)
- new net MDI1-: T1.8, U5.5 (MDIN1)
- new net MDI2+: T2.1, U7.2 (MDIP0)
- new net MDI2-: T2.3, U7.3 (MDIN0)
- new net MDI3+: T2.6, U7.4 (MDIP1)
- new net MDI3-: T2.8, U7.5 (MDIN1)
- new net VBUS: C1.1, C10.1, C11.1, C2.1, C3.1, C4.1, C5.1, C6.1, C8.1, TP24.1, U1.19 (V5), U2.6 (VIN), U3.A4B9 (VBUS), U3.B4A9 (VBUS)
Other:
- company: (none) -> Hack Club
- title: (none) -> tobycm's usb hub

Commit message: PCB done!!!
Parts:
- removed RJ1, RJ2: X12ADGWA3DY1027, easyeda2kicad:RJ45-TH_XKB_X12ADHWA3DY1027, symbol easyeda2kicad:X12ADGWA3DY1027
- removed TP10, TP9: TestPoint, TestPoint:TestPoint_Pad_D2.0mm, symbol Connector:TestPoint
- added C41, C42: 1n, Capacitor_SMD:C_1206_3216Metric, symbol Device:C
- added H1, H2, H3: MountingHole, MountingHole:MountingHole_3.2mm_M3_Pad, symbol Mechanical:MountingHole
- added R10, R11, R12, R13, R14, R15, R8, R9: 75, Resistor_SMD:R_0402_1005Metric, symbol Device:R
- added R16, R17, R18, R19: 470, Resistor_SMD:R_0402_1005Metric, symbol Device:R
- added R6, R7: 5.1k, Resistor_SMD:R_0402_1005Metric, symbol Device:R
- added RJ1, RJ2: R-RJ45S08P-C000, easyeda2kicad:RJ45-TH_R-RJ45S08P-C000, symbol easyeda2kicad:R-RJ45S08P-C000
- C37, C38, C39, C40: LCSC Part # C1525 -> C60133
- TP1, TP11, TP12, TP13, TP14, TP15, TP16, TP17, TP18, TP19, TP2, TP20, TP21, TP22, TP23, TP24, TP25, TP26, TP28, TP3, TP30, TP33, TP35, TP36, TP4, TP5, TP6, TP7, TP8: footprint TestPoint:TestPoint_Pad_D2.0mm -> TestPoint:TestPoint_Pad_D1.0mm
- TP27: footprint TestPoint:TestPoint_Pad_D2.0mm -> TestPoint:TestPoint_Pad_D1.0mm; now not fitted
Connections:
- net GND: now also R6.2, R7.2
- net LED0: now also RJ1.10 (Y-)
- net LED1: now also RJ1.12 (G-)
- net LED2: now also RJ2.10 (Y-)
- net LED3: now also RJ2.12 (G-)
- net MDI0+: now also T1.8; no longer T1.1
- net MDI0-: now also T1.6; no longer T1.3
- net MDI1+: now also T1.3; no longer T1.6
- net MDI1-: now also T1.1; no longer T1.8
- net MDI2+: now also T2.8; no longer T2.1
- net MDI2-: now also T2.6; no longer T2.3
- net MDI3+: now also T2.3; no longer T2.6
- net MDI3-: now also T2.1; no longer T2.8
- net at C40.1, T2.7: no longer C39.1, T2.2
- net TDI1-: now reaches T1.16
- net TDI1-: now also RJ1.6
- net TDI1+: now reaches T1.14
- net TDI1+: now also RJ1.3
- net TDI0+: now reaches T1.11
- net TDI0+: now also RJ1.1
- net TDI0-: now reaches T1.9
- net TDI0-: now also RJ1.2
- net at C37.1, T1.2: no longer C38.1, T1.7
- net TDI3-: now reaches T2.16
- net TDI3-: now also RJ2.6
- net TDI3+: now reaches T2.14
- net TDI3+: now also RJ2.3
- net TDI2+: now reaches T2.11
- net TDI2+: now also RJ2.1
- net TDI2-: now reaches T2.9
- net TDI2-: now also RJ2.2
- net at T2.10: now also R13.2
- net at T2.15: now also R12.2
- net at U3.A5 (CC1): now also R6.1
- net at U3.B5 (CC2): now also R7.1
- net at T1.10: now also R9.2
- net at T1.15: now also R8.2
- net +1V0: no longer names the net of C26.1, C27.1, U7.16 (DVDD10), U7.23 (AVDD10), U7.9 (U2VDD10)
- net +1V0: no longer C20.1, C21.1, U5.16 (DVDD10), U5.23 (AVDD10), U5.9 (U2VDD10)
- net +1V1: no longer names the net of C22.1, C23.1, U5.12 (DVDD10_UPS)
- net +1V1: no longer C30.1, C31.1, U7.12 (DVDD10_UPS)
- net +3.3V renamed +3.3V2
- net +3.3V2: now also R16.1, R17.1; no longer R4.1, U7.1 (AVDD33), U7.10 (AVDD33), U7.13 (DVDD33)
- new net: C20.1, C21.1, U5.16 (DVDD10), U5.23 (AVDD10), U5.9 (U2VDD10)
- new net: R18.2, RJ2.9 (Y+)
- new net: R17.2, RJ1.11 (G+)
- new net: R10.1, RJ1.4, RJ1.5
- new net: R11.1, RJ1.7, RJ1.8
- new net: R16.2, RJ1.9 (Y+)
- new net: C42.1, R12.1, R13.1, R14.2, R15.2
- new net: C41.1, R10.2, R11.2, R8.1, R9.1
- new net: C30.1, C31.1, U7.12 (DVDD10_UPS)
- new net: R14.1, RJ2.4, RJ2.5
- new net: R19.2, RJ2.11 (G+)
- new net: R15.1, RJ2.7, RJ2.8
- new net: C39.1, T2.2
- new net: C38.1, T1.7
- new net +3.3V3: R18.1, R19.1, R4.1, U7.1 (AVDD33), U7.10 (AVDD33), U7.13 (DVDD33)
- new net GND2: C41.2, RJ1.13 (S), RJ1.14 (S)
- new net GND3: C42.2, RJ2.13 (S), RJ2.14 (S)
Other:
- moved on the sheet: C18, C19, C20, C21, C22, C23, C26, C27, C28, C29, C30, C31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
