File: pcb/skibidi-usb-hub.kicad_pcb (KiCad board)
At the start: 4 copper layers, 50 x 65 mm, 115 parts, among them SW1 B3U-1100PM, SW2 B3U-1100PM, T1 H1102NLT_C20623173, T2 H1102NLT_C20623173, U1 CH334F_C5187527, U10 PJ-320A-4P DIP, U2 CH217K, U3 GT-USB-7010ASV, U4 GT-USB-7010ASV, U5 RTL8152B-VB-CG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

Commit message: add EMI capacitor for ethernet chassis ground and logic ground
Signed-off-by: Toby Cm <toby@vsus.app>
Parts:
- added C43: 1n, Capacitor_SMD:C_1206_3216Metric, F.Cu at (134.0, 63.0)
- added C44: 1n, Capacitor_SMD:C_1206_3216Metric, F.Cu at (134.8, 104.2)
- moved TP24 2.83 mm to (136.2, 63.2)
- moved C42 0.25 mm to (138.2, 102.5)
Routing:
- net VBUS: track 76.5 -> 73.7 mm
- net GND: track 99.2 -> 101.9 mm, vias 64 -> 66
- net Net-(C42-Pad1): track 7.97 -> 5.87 mm
- net +5V: vias 57 -> 61
