File: pcb/skibidi-usb-hub.kicad_sch (KiCad schematic)
At the start: 116 parts, among them SW1 B3U-1100PM, SW2 B3U-1100PM, T1 H1102NLT_C20623173, T2 H1102NLT_C20623173, U1 CH334F_C5187527, U10 PJ-320A-4P DIP, U2 CH217K, U3 GT-USB-7010ASV, U4 GT-USB-7010ASV, U5 RTL8152B-VB-CG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

Commit message: add EMI capacitor for ethernet chassis ground and logic ground
Signed-off-by: Toby Cm <toby@vsus.app>
Parts:
- added C43, C44: 1n, Capacitor_SMD:C_1206_3216Metric, symbol Device:C
Connections:
- net GND: now also C43.1, C44.1
- net GND2: now also C43.2
- net GND3: now also C44.2
